File: hardware/matrix64x8/matrix64x8.kicad_sch (KiCad schematic)
At the start: 61 parts, among them J0 LED Matrix, J0 POWER, J1 Discrete LEDs, J1 LED Matrix, J2 Discrete LEDs, J2 POWER, J3 Remove to program, Q0 FQP47P06, U0 74HCT238, U1 ULN2803A, U2 ULN2803A, U3 TPIC6B595

Commit message: hw 2.0
Parts:
- removed JP?: Short to Cascade, symbol Jumper:Jumper_2_Open
- removed U3: TPIC6B595, symbol Interface_Expansion:TPIC6595
- added C1_{SH}: 0.1µF, symbol Device:C
- added J3_{SH}: RS-485, symbol Connector:Screw_Terminal_01x03
- added J?: Conn_01x08_Pin, symbol Connector:Conn_01x08_Pin
- added R0_{SH}: 10K, symbol Device:R_US
- added U0_{SH}: THVD1439, Package_SO:SOIC-8_3.9x4.9mm_P1.27mm, symbol Interface_UART:THVD1420D
- added U3: TPIC6C595, symbol local:TPIC6595
- renumbered R72 to R24, R73 to R25, R74 to R26, R75 to R27, R76 to R28, R77 to R29, R78 to R30, R79 to R31, R15 to R9
Connections:
- net +5V: now also C1_{SH}.1, U0_{SH}.8 (VCC), U3.1 (VCC)
- net GNDREF: now also C1_{SH}.2, J3_{SH}.3 (Pin_3), R0_{SH}.2, U0_{SH}.5 (GND), U3.16 (GND)
- net RCLK: now also U3.10 (RCLK)
- net SRCLK: now also U3.15 (SRCK)
- net ~{G}: now also U3.8 (~{G})
- net ~{SRCLR}: now also U3.7 (~{SRCLR})
- net at R8.1: now also U3.3 (DRAIN0)
- net at R9.1: now also U3.14 (DRAIN7)
- net at R12.1: now also U3.11 (DRAIN4)
- net at R13.1: now also U3.12 (DRAIN5)
- net at R14.1: now also U3.13 (DRAIN6)
- net at J1.12 (Pin_12): now also U3.2 (SER_IN)
- net at R9.1: now also U3.4 (DRAIN1)
- net at R10.1: now also U3.5 (DRAIN2)
- net at R11.1: now also U3.6 (DRAIN3)
- new net: J?.2 (Pin_2), U0_{SH}.1 (RO)
- new net: R0_{SH}.1, U0_{SH}.2 (~{RE}), U0_{SH}.3 (DE)
- new net: J?.1 (Pin_1), U0_{SH}.4 (DI)
- new net: J3_{SH}.2 (Pin_2), U0_{SH}.6 (A)
- new net: J3_{SH}.1 (Pin_1), U0_{SH}.7 (B)
- no-connect marks 15 -> 21
Other:
- note added: "01-SEP-2023"
- note added: "16"
- note added: "17"
- note added: "18"
- note added: "19"
- note added: "2.0.0"
- note added: "20"
- note added: "21"
- note added: "A"
- note added: "B"
- note added: "R24-R31 as appropriate for each LED value."
- note added: "R8-R23 as appropriate to limit LED current."
- note added: "Repeat for total of 8 blocks with U3-U10, C1-C8, R8-R23, with inputs D_{1}-D_{7}, outputs to columns 0-63."
- note added: "Rx 15"
- note added: "Tx 14"
- note added: "UART3"
- note removed: "09-AUG-2023"
- note removed: "1.0.1"
- note removed: "R72-R79 as appropriate for each LED value."
- note removed: "R8-R71 as appropriate to limit LED current."
- note removed: "Repeat for total of 8 blocks with U3-U10, C1-C8, R8-R71, with inputs D_{1}-D_{7}, outputs to columns 0-63."
- moved on the sheet: J0, J1

Commit message: typo
Connections:
- net at R0_{SH}.1, U0_{SH}.2 (~{RE}), U0_{SH}.3 (DE): now also J?.8 (Pin_8)
- no-connect marks 21 -> 20
Other:
- note added: "A (D+)"
- note added: "B (D-)"
- note added: "To U4-U10 pin 2 for D_{1}-D_{7} respectively."
- note added: "~{RE}/DE"
- note removed: "A"
- note removed: "B"
- note removed: "To U4-U10 pin 3 for D1-D7 respectively."
Changed lines of the file:
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@@
   (junction (at 93.98 157.48) (diameter 0) (color 0 0 0 0)
   )
-  (junction (at 145.415 255.27) (diameter 0) (color 0 0 0 0)
-  )
   (junction (at 295.275 93.345) (diameter 0) (color 0 0 0 0)
   )
@@
   (junction (at 246.38 142.24) (diameter 0) (color 0 0 0 0)
   )
-  (no_connect (at 95.25 199.39))
+  (junction (at 108.585 238.76) (diameter 0) (color 0 0 0 0)
+  )
   (no_connect (at 95.25 191.77))
   (no_connect (at 34.925 210.185))
@@
     (stroke (width 0) (type default))
   )
-  (wire (pts (xy 108.585 233.045) (xy 108.585 236.22))
+  (wire (pts (xy 118.745 233.045) (xy 118.745 236.22))
     (stroke (width 0) (type default))
   )
@@
     (stroke (width 0) (type dash))
   )
-  (wire (pts (xy 95.885 233.045) (xy 108.585 233.045))
+  (wire (pts (xy 95.885 233.045) (xy 118.745 233.045))
     (stroke (width 0) (type default))
   )
@@
     (stroke (width 0) (type dash))
   )
-  (wire (pts (xy 145.415 230.505) (xy 145.415 255.27))
-    (stroke (width 0) (type default))
-  )
   (wire (pts (xy 149.86 73.66) (xy 154.305 73.66))
     (stroke (width 0) (type default))
@@
     (stroke (width 0) (type default))
   )
-  (wire (pts (xy 118.745 236.22) (xy 108.585 236.22))
-    (stroke (width 0) (type default))
-  )
   (wire (pts (xy 203.835 216.535) (xy 212.09 216.535))
     (stroke (width 0) (type default))
@@
     (stroke (width 0) (type default))
   )
+  (wire (pts (xy 95.25 199.39) (xy 100.965 199.39))
+    (stroke (width 0) (type default))
+  )
   (wire (pts (xy 69.215 76.2) (xy 71.755 76.2))
     (stroke (width 0) (type default))
@@
     (stroke (width 0) (type default))
   )
-  (wire (pts (xy 145.415 255.27) (xy 151.13 255.27))
+  (wire (pts (xy 128.905 255.27) (xy 151.13 255.27))
     (stroke (width 0) (type default))
   )
@@
     (stroke (width 0) (type default))
   )
+  (wire (pts (xy 100.965 199.39) (xy 100.965 238.76))
+    (stroke (width 0) (type default))
+  )
   (wire (pts (xy 66.04 71.12) (xy 71.755 71.12))
     (stroke (width 0) (type default))
@@
     (stroke (width 0) (type default))
   )
-  (wire (pts (xy 128.905 255.27) (xy 145.415 255.27))
+  (wire (pts (xy 100.965 238.76) (xy 108.585 238.76))
     (stroke (width 0) (type default))
   )
@@
     (effects (font (size 1.27 1.27)) (justify right bottom))
   )
-  (text "To U4-U10 pin 3 for\nD1-D7 respectively." (at 83.185 47.625 0)
+  (text "To U4-U10 pin 2 for\nD_{1}-D_{7} respectively." (at 83.185 47.625 0)
     (effects (font (size 1.27 1.27)) (justify left bottom))
   )
@@
     (effects (font (size 1.27 1.27)) (justify left bottom))
   )
-  (text "B" (at 158.75 237.49 0)
+  (text "B (D-)" (at 158.75 237.49 0)
     (effects (font (size 1.27 1.27)) (justify left bottom))
   )
@@
     (effects (font (size 1.27 1.27)) (justify left bottom))
   )
-  (text "A" (at 158.75 240.03 0)
+  (text "A (D+)" (at 158.75 240.03 0)
     (effects (font (size 1.27 1.27)) (justify left bottom))
   )
@@
     (effects (font (size 1.27 1.27)) (justify left bottom))
   )
+  (text "~{RE}/DE" (at 100.33 219.71 90)
+    (effects (font (size 1.27 1.27)) (justify left bottom))
+  )
   (text "D_{3}" (at 207.01 208.915 0)
     (effects (font (size 1.27 1.27)) (justify left bottom))
@@
         )
       )
+    )
+  )
+  (symbol (lib_id "power:GNDREF") (at 145.415 230.505 0) (unit 1)
+    (in_bom yes) (on_board yes) (dnp no) (fields_autoplaced)
+    (property "Reference" "#PWR030" (at 145.415 236.855 0)
+      (effects (font (size 1.27 1.27)) hide)
+    )
+    (property "Value" "GNDREF" (at 145.415 234.95 0)
+      (effects (font (size 1.27 1.27)) hide)
+    )
+    (property "Footprint" "" (at 145.415 230.505 0)
+      (effects (font (size 1.27 1.27)) hide)
+    )
+    (property "Datasheet" "" (at 145.415 230.505 0)
+      (effects (font (size 1.27 1.27)) hide)
+    )
+    (pin "1")
+    (instances
+      (project "matrix64x8"
+        (path "/68206880-187a-441b-ad1d-285a8d6fa444"
+          (reference "#PWR030") (unit 1)
+        )
+      )

Commit message: updated boards
Parts:
- added C0: 0.1µF, symbol Device:C
- added J3: Termination, symbol Jumper:Jumper_2_Bridged
- added R1_{SH}: 120Ω, symbol Device:R_US
- renumbered J3_{SH} to J4_{SH}
Connections:
- net +5V: now also C0.1
- net GNDREF: now also C0.2
- net at J4_{SH}.2 (Pin_2), U0_{SH}.6 (A): now also J3.2 (B)
- net at J4_{SH}.1 (Pin_1), U0_{SH}.7 (B): now also R1_{SH}.1
- new net: J3.1 (A), R1_{SH}.2
Other:
- moved on the sheet: J4_{SH}
Changed lines of the file:
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@@
   (junction (at 205.74 221.615) (diameter 0) (color 0 0 0 0)
   )
+  (junction (at 144.78 236.22) (diameter 0) (color 0 0 0 0)
+  )
   (junction (at 86.995 76.2) (diameter 0) (color 0 0 0 0)
   )
@@
   (junction (at 93.98 157.48) (diameter 0) (color 0 0 0 0)
   )
+  (junction (at 144.78 254) (diameter 0) (color 0 0 0 0)
+  )
   (junction (at 295.275 93.345) (diameter 0) (color 0 0 0 0)
   )
@@
   (junction (at 323.85 86.995) (diameter 0) (color 0 0 0 0)
   )
+  (junction (at 106.045 122.555) (diameter 0) (color 0 0 0 0)
+  )
   (junction (at 323.85 74.295) (diameter 0) (color 0 0 0 0)
   )
@@
     (stroke (width 0) (type default))
   )
+  (wire (pts (xy 144.78 236.22) (xy 157.48 236.22))
+    (stroke (width 0) (type default))
+  )
   (wire (pts (xy 170.18 211.455) (xy 191.135 211.455))
     (stroke (width 0) (type default))
@@
     (stroke (width 0) (type dash))
   )
+  (wire (pts (xy 106.045 122.555) (xy 116.205 122.555))
+    (stroke (width 0) (type default))
+  )
   (wire (pts (xy 95.25 201.93) (xy 111.125 201.93))
     (stroke (width 0) (type default))
@@
     (stroke (width 0) (type default))
   )
-  (wire (pts (xy 139.065 236.22) (xy 151.13 236.22))
+  (wire (pts (xy 139.065 236.22) (xy 144.78 236.22))
     (stroke (width 0) (type default))
   )
@@
     (stroke (width 0) (type default))
   )
-  (wire (pts (xy 139.065 243.84) (xy 139.065 238.76))
-    (stroke (width 0) (type default))
-  )
   (wire (pts (xy 212.09 198.755) (xy 181.61 198.755))
     (stroke (width 0) (type default))
@@
     (stroke (width 0) (type default))
   )
-  (wire (pts (xy 139.065 238.76) (xy 151.13 238.76))
-    (stroke (width 0) (type default))
-  )
   (wire (pts (xy 138.43 196.85) (xy 133.985 196.85))
     (stroke (width 0) (type default))
@@
     (stroke (width 0) (type default))
   )
+  (wire (pts (xy 157.48 238.76) (xy 154.305 238.76))
+    (stroke (width 0) (type default))
+  )
   (wire (pts (xy 69.215 58.42) (xy 69.215 52.705))
     (stroke (width 0) (type default))
@@
     (stroke (width 0) (type default))
   )
+  (wire (pts (xy 139.065 254) (xy 139.065 243.84))
+    (stroke (width 0) (type default))
+  )
   (wire (pts (xy 106.045 165.1) (xy 106.045 166.37))
     (stroke (width 0) (type default))
@@
     (stroke (width 0) (type default))
   )
-  (wire (pts (xy 128.905 255.27) (xy 151.13 255.27))
+  (wire (pts (xy 128.905 255.27) (xy 157.48 255.27))
     (stroke (width 0) (type default))
   )
@@
     (stroke (width 0) (type default))
   )
+  (wire (pts (xy 154.305 254) (xy 144.78 254))
+    (stroke (width 0) (type default))
+  )
   (wire (pts (xy 137.16 48.895) (xy 137.16 66.04))
     (stroke (width 0) (type default))
@@
     (stroke (width 0) (type default))
   )
+  (wire (pts (xy 106.045 122.555) (xy 106.045 137.16))
+    (stroke (width 0) (type default))
+  )
   (wire (pts (xy 265.43 74.295) (xy 265.43 86.995))
     (stroke (width 0) (type default))
@@
     (stroke (width 0) (type default))
   )
+  (wire (pts (xy 154.305 238.76) (xy 154.305 254))
+    (stroke (width 0) (type default))
+  )
   (wire (pts (xy 84.455 81.28) (xy 86.995 81.28))
     (stroke (width 0) (type default))
@@
     (stroke (width 0) (type default))
   )
-  (wire (pts (xy 106.045 130.81) (xy 106.045 137.16))
+  (wire (pts (xy 106.045 119.38) (xy 106.045 122.555))
     (stroke (width 0) (type default))
   )
@@
     (stroke (width 0) (type default))
   )
-  (wire (pts (xy 151.13 241.3) (xy 151.13 255.27))
+  (wire (pts (xy 144.78 254) (xy 139.065 254))
+    (stroke (width 0) (type default))
+  )
+  (wire (pts (xy 157.48 241.3) (xy 157.48 255.27))
     (stroke (width 0) (type default))
   )
@@
     (effects (font (size 1.27 1.27)) (justify left bottom))
   )
-  (text "B (D-)" (at 158.75 237.49 0)
+  (text "B (D-)" (at 165.1 237.49 0)
     (effects (font (size 1.27 1.27)) (justify left bottom))
   )
@@
     (effects (font (size 1.27 1.27)) (justify left bottom))
   )
-  (text "A (D+)" (at 158.75 240.03 0)
+  (text "A (D+)" (at 165.1 240.03 0)
     (effects (font (size 1.27 1.27)) (justify left bottom))
   )
@@
     (effects (font (size 1.27 1.27)) (justify right bottom))
   )
-  (text "GND" (at 158.75 242.57 0)
+  (text "GND" (at 165.1 242.57 0)
     (effects (font (size 1.27 1.27)) (justify left bottom))
   )
@@
     )
   )
+  (symbol (lib_id "Device:C") (at 116.205 126.365 0) (unit 1)
+    (in_bom yes) (on_board yes) (dnp no) (fields_autoplaced)
+    (property "Reference" "C0" (at 119.38 125.095 0)
+      (effects (font (size 1.27 1.27)) (justify left))
+    )
+    (property "Value" "0.1µF" (at 119.38 127.635 0)
+      (effects (font (size 1.27 1.27)) (justify left))
+    )
+    (property "Footprint" "" (at 117.1702 130.175 0)
+      (effects (font (size 1.27 1.27)) hide)
+    )
+    (property "Datasheet" "~" (at 116.205 126.365 0)
+      (effects (font (size 1.27 1.27)) hide)
+    )
+    (pin "1")
+    (pin "2")
+    (instances
+      (project "matrix64x8"
+        (path "/68206880-187a-441b-ad1d-285a8d6fa444"
+          (reference "C0") (unit 1)
+        )
+      )
+    )
+  )
   (symbol (lib_id "Device:LED") (at 272.415 74.295 0) (unit 1)
     (in_bom yes) (on_board yes) (dnp no) (fields_autoplaced)
@@
     )
   )
-  (symbol (lib_id "Connector:Screw_Terminal_01x03") (at 156.21 238.76 0) (unit 1)
+  (symbol (lib_id "Connector:Screw_Terminal_01x03") (at 162.56 238.76 0) (unit 1)
     (in_bom yes) (on_board yes) (dnp no)
-    (property "Reference" "J3_{SH}" (at 155.575 229.87 0)
+    (property "Reference" "J4_{SH}" (at 161.925 229.87 0)
       (effects (font (size 1.27 1.27)) (justify left))
     )
-    (property "Value" "RS-485" (at 155.575 232.41 0)
+    (property "Value" "RS-485" (at 161.925 232.41 0)
       (effects (font (size 1.27 1.27)) (justify left))
     )
-    (property "Footprint" "" (at 156.21 238.76 0)
+    (property "Footprint" "" (at 162.56 238.76 0)
       (effects (font (size 1.27 1.27)) hide)
     )
-    (property "Datasheet" "~" (at 156.21 238.76 0)
+    (property "Datasheet" "~" (at 162.56 238.76 0)
       (effects (font (size 1.27 1.27)) hide)
     )
@@
       (project "matrix64x8"
         (path "/68206880-187a-441b-ad1d-285a8d6fa444"
-          (reference "J3_{SH}") (unit 1)
+          (reference "J4_{SH}") (unit 1)
         )
       )
@@
     )
   )
-  (symbol (lib_id "power:+5V") (at 106.045 130.81 0) (unit 1)
+  (symbol (lib_id "power:+5V") (at 106.045 119.38 0) (unit 1)
     (in_bom yes) (on_board yes) (dnp no)
-    (property "Reference" "#PWR012" (at 106.045 134.62 0)
+    (property "Reference" "#PWR012" (at 106.045 123.19 0)
       (effects (font (size 1.27 1.27)) hide)
     )
-    (property "Value" "+5V" (at 106.045 125.73 0)
+    (property "Value" "+5V" (at 106.045 114.3 0)
       (effects (font (size 1.27 1.27)))
     )
-    (property "Footprint" "" (at 106.045 130.81 0)
+    (property "Footprint" "" (at 106.045 119.38 0)
       (effects (font (size 1.27 1.27)) hide)
     )
-    (property "Datasheet" "" (at 106.045 130.81 0)
+    (property "Datasheet" "" (at 106.045 119.38 0)
       (effects (font (size 1.27 1.27)) hide)
     )
@@
     )
   )
+  (symbol (lib_id "Device:R_US") (at 144.78 240.03 0) (unit 1)
+    (in_bom yes) (on_board yes) (dnp no)
+    (property "Reference" "R1_{SH}" (at 146.685 238.76 0)
+      (effects (font (size 1.27 1.27)) (justify left))
+    )
+    (property "Value" "120Ω" (at 146.685 241.3 0)
+      (effects (font (size 1.27 1.27)) (justify left))
+    )
+    (property "Footprint" "" (at 145.796 240.284 90)
+      (effects (font (size 1.27 1.27)) hide)
+    )
+    (property "Datasheet" "~" (at 144.78 240.03 0)
+      (effects (font (size 1.27 1.27)) hide)
+    )
+    (pin "1")
+    (pin "2")
+    (instances
+      (project "matrix64x8"
+        (path "/68206880-187a-441b-ad1d-285a8d6fa444"
+          (reference "R1_{SH}") (unit 1)
+        )
+      )
+    )
+  )
   (symbol (lib_id "power:GNDREF") (at 135.255 167.64 0) (unit 1)
     (in_bom yes) (on_board yes) (dnp no) (fields_autoplaced)
@@
     )
   )
+  (symbol (lib_id "power:GNDREF") (at 116.205 130.175 0) (unit 1)
+    (in_bom yes) (on_board yes) (dnp no) (fields_autoplaced)
+    (property "Reference" "#PWR031" (at 116.205 136.525 0)
+      (effects (font (size 1.27 1.27)) hide)
+    )
+    (property "Value" "GNDREF" (at 116.205 135.255 0)
+      (effects (font (size 1.27 1.27)) hide)
+    )
+    (property "Footprint" "" (at 116.205 130.175 0)
+      (effects (font (size 1.27 1.27)) hide)
+    )
+    (property "Datasheet" "" (at 116.205 130.175 0)
+      (effects (font (size 1.27 1.27)) hide)
+    )
+    (pin "1")
+    (instances
+      (project "matrix64x8"
+        (path "/68206880-187a-441b-ad1d-285a8d6fa444"
+          (reference "#PWR031") (unit 1)
+        )
+      )
+    )
+  )
   (symbol (lib_id "power:GNDREF") (at 128.905 255.27 0) (unit 1)
     (in_bom yes) (on_board yes) (dnp no) (fields_autoplaced)
@@
         )
       )
+    )
+  )
+  (symbol (lib_id "Jumper:Jumper_2_Bridged") (at 144.78 248.92 270) (unit 1)
+    (in_bom yes) (on_board yes) (dnp no)
+    (property "Reference" "J3" (at 146.685 246.38 0)
+      (effects (font (size 1.27 1.27)) (justify left))
+    )
+    (property "Value" "Termination" (at 142.875 242.57 0)
+      (effects (font (size 1.27 1.27)) (justify left))
+    )
+    (property "Footprint" "" (at 144.78 248.92 0)
+      (effects (font (size 1.27 1.27)) hide)
+    )
+    (property "Datasheet" "~" (at 144.78 248.92 0)
+      (effects (font (size 1.27 1.27)) hide)
+    )
+    (pin "1")
+    (pin "2")
+    (instances
+      (project "matrix64x8shield"
+        (path "/464f095f-bee4-4d28-b0df-0d48998e6d23"
+          (reference "J3") (unit 1)
+        )
+      )
+      (project "matrix64x8"
+        (path "/68206880-187a-441b-ad1d-285a8d6fa444"
+          (reference "J5_{SH}") (unit 1)
+        )
+      )

Commit message: bom
Parts:
- removed J2: POWER, symbol Connector:Screw_Terminal_01x04
- removed J4_{SH}: RS-485, symbol Connector:Screw_Terminal_01x03
- added J2_{SH}: POWER, symbol Connector:Screw_Terminal_01x05
- added J4_{SH}: RS-485, symbol Connector:Screw_Terminal_01x06
- U2: value ULN2803A -> ULN2803A*
Connections:
- net +5V: now also J2_{SH}.1 (Pin_1)
- net GNDREF: now also J2_{SH}.2 (Pin_2), J2_{SH}.3 (Pin_3), J4_{SH}.3 (Pin_3), J4_{SH}.4 (Pin_4)
- net at J3.2 (B), U0_{SH}.6 (A): now also J4_{SH}.2 (Pin_2), J4_{SH}.6 (Pin_6)
- net at R1_{SH}.1, U0_{SH}.7 (B): now also J4_{SH}.1 (Pin_1), J4_{SH}.5 (Pin_5)
- net at J?.8 (Pin_8): now also J2_{SH}.4 (Pin_4), J2_{SH}.5 (Pin_5)
Other:
- note added: "*May substitute ULN2803C for ULN2803A. The pinouts are compatible except the 2803C has two extra pins at the bottom (10 & 11) which are not connected to anything."
- note added: "1"
- note added: "A (D+ IN)"
- note added: "A (D+ OUT)"
- note added: "B (D- IN)"
- note added: "B (D- OUT)"
- note added: "Repeat for a total of 8 outputs for R0-R7, Q0-Q7, from pins 18-11 respectively, driving rows 0-7."
- note removed: "A (D+)"
- note removed: "B (D-)"
- note removed: "Repeat for total of 8 outputs for R0-R7, Q0-Q7, from pins 17-11 respectively, driving rows 0-7."
