File: hardware/busylight/busylight.kicad_sch (KiCad schematic)
At the start: 0 parts

Commit message: wip
Parts:
- added A0: Sparkfun_Pro_Micro, symbol MCU_Module_Local:Sparkfun_Pro_Micro
- added C0: 0.1μF, symbol Device:C
- added D_{x}0, D_{x}1, D_{x}2, D_{x}3, D_{x}4, D_{x}5, D_{x}6, D_{x}7: LED, symbol Device:LED
- added J0: LED TREE, symbol Connector:DIN-8
- added J1: RS-485, symbol Connector:Screw_Terminal_01x16
- added J2: To pin of J0, symbol Connector:Conn_01x01_Pin
- added R0, R1, R2: 10K, symbol Device:R_US
- added R_{term}: 120Ω, symbol Device:R_US
- added Rx0*, Rx1*: R_Network04, Resistor_THT:R_Array_SIP5, symbol Device:R_Network04
- added U0: ULN2003A, symbol Transistor_Array:ULN2003A
- added U1: THVD1439, Package_SO:SOIC-8_3.9x4.9mm_P1.27mm, symbol Interface_UART:THVD1420D
Connections:
- new net: A0.5 (D2), R2.1, U1.3 (DE)
- new net: J0.1, U0.10 (O7)
- new net: J0.2, U0.12 (O5)
- new net: J0.3, U0.13 (O4)
- new net: J0.4, U0.11 (O6)
- new net: J0.5, U0.14 (O3)
- new net: J0.6, U0.16 (O1)
- new net: J0.8, U0.15 (O2)
- new net: J2.1 (Pin_1), Rx0*.1 (common), Rx1*.1 (common)
- new net: D_{x}3.1 (K), Rx0*.2 (R1)
- new net: D_{x}2.1 (K), Rx0*.3 (R2)
- new net: D_{x}1.1 (K), Rx0*.4 (R3)
- new net: D_{x}0.1 (K), Rx0*.5 (R4)
- new net: D_{x}7.1 (K), Rx1*.2 (R1)
- new net: J1.1 (Pin_1), J1.2 (Pin_2)
- new net: J1.10 (Pin_10), J1.12 (Pin_12), U1.7 (B)
- new net: J1.11 (Pin_11), J1.9 (Pin_9), U1.6 (A)
- new net: A0.24 (RAW), J1.15 (Pin_15), J1.16 (Pin_16)
- new net: J1.3 (Pin_3), J1.4 (Pin_4)
- new net: J1.5 (Pin_5), J1.6 (Pin_6)
- new net: D_{x}4.1 (K), Rx1*.5 (R4)
- new net: D_{x}5.1 (K), Rx1*.4 (R3)
- new net: D_{x}6.1 (K), Rx1*.3 (R2)
- new net: A0.1 (D1/TX), U1.4 (DI)
- new net: A0.10 (D7), U0.7 (I7)
- new net: A0.11 (D8), U0.6 (I6)
- new net: A0.12 (D9~), U0.5 (I5)
- new net: A0.13 (D10), U0.3 (I3)
- new net: A0.14 (D16/MOSI), U0.2 (I2)
- new net: A0.15 (D14/MISO), U0.1 (I1)
- new net: A0.2 (D0/RX), R0.2, U1.1 (RO)
- new net: A0.6 (D3~), R1.2, U1.2 (~{RE})
- new net: A0.9 (D6~), U0.4 (I4)
- new net +5V: A0.21 (Vcc), C0.1, D_{x}0.2 (A), D_{x}1.2 (A), D_{x}2.2 (A), D_{x}3.2 (A), D_{x}4.2 (A), D_{x}5.2 (A), D_{x}6.2 (A), D_{x}7.2 (A), J0.7, R0.1, R1.1, U1.8 (VCC)
- new net Earth: A0.23 (GND), A0.3 (GND), A0.4 (GND), C0.2, J1.13 (Pin_13), J1.14 (Pin_14), J1.7 (Pin_7), J1.8 (Pin_8), R2.2, U0.8 (GND), U1.5 (GND)
- no-connect marks 0 -> 9
Other:
- note added: "*R value chosen as appropriate for the LEDs used and supply voltage."
- note added: "2.1.0"
- note added: "27-Sep-2024"
- note added: "8-PIN CAT6 CABLES A (IN) AND B (OUT)"
- note added: "A1 RDATA A(+) IN"
- note added: "A2 RDATA B(-) IN"
- note added: "A3 CC+ IN / +9V POWER SUPPLY"
- note added: "A4 DATA B(-) IN"
- note added: "A5 DATA A(+) IN"
- note added: "A6 CCr IN"
- note added: "A7 GND"
- note added: "A8 GND"
- note added: "B1 RDATA A(+) OUT"
- note added: "B2 RDATA B(-) OUT"
- note added: "B3 CC+ OUT"
- note added: "B4 DATA B(-) OUT"
- note added: "B5 DATA A(+) OUT"
- note added: "B6 CCr OUT"
- note added: "B7 GND"
- note added: "B8 GND"
- note added: "BUSYLIGHT SHIELD"
- note added: "Busylight Shield"
- note added: "Copyright 2021, 2024 Steven Willoughby * Open-source hardware Under BSD 3-clause license."
- note added: "EACH LED TREE LEVEL"
- note added: "L_{0} GREEN"
- note added: "L_{1} AMBER"
- note added: "L_{2} AMBER"
- note added: "L_{3} RED"
- note added: "L_{4} RED"
- note added: "L_{5} BLUE"
- note added: "L_{6} BLUE"
- note added: "Powered via USB connector on Pro Micro board or external supply on "RAW" (which runs through the internal 5V regulator on the Pro Micro)."
- note added: "Terminator"
- note added: "To pin 7 of J0"

Commit message: design updates
Parts:
- added C1: 100μF, symbol Device:C_Polarized_Small_US
- added D0: 1A, symbol Device:D_Filled
- added J3: SPEAKER, symbol Connector:Screw_Terminal_01x02
- added LS1: Speaker, symbol Device:Speaker
- added Q0: BC547 or 2N2222, Package_TO_SOT_THT:TO-92_Inline, symbol Transistor_BJT:BC547
- added R3: 10K, symbol Device:R_US
Connections:
- net +5V: now also J3.1 (Pin_1)
- net Earth: now also Q0.3 (E)
- net at J1.15 (Pin_15), J1.16 (Pin_16): now also D0.2 (A); no longer A0.24 (RAW)
- net at A0.8 (D5~): now also C1.2
- new net: A0.24 (RAW), D0.1 (K)
- new net: J3.2 (Pin_2), Q0.1 (C), R3.1
- new net: C1.1, Q0.2 (B), R3.2
- no-connect marks 9 -> 8
Other:
- note added: "09-Oct-2024"
- note added: "2.2.0"
- note removed: "2.1.0"
- note removed: "27-Sep-2024"

Commit message: tweaks
Parts:
- added R4: 10K, symbol Device:R_US
Connections:
- net at C1.2: now also R4.1; no longer A0.8 (D5~)
- new net: A0.8 (D5~), R4.2
Other:
- note added: "Optional series resistor (or jumper wire)"
Changed lines of the file:
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@@
+	(wire
+		(pts
+			(xy 78.74 119.38) (xy 78.74 78.74)
+		)
+		(stroke
+			(width 0)
+			(type default)
+		)
+	)
 	(wire
 		(pts
@@
 	(wire
 		(pts
-			(xy 78.74 147.32) (xy 78.74 78.74)
+			(xy 78.74 147.32) (xy 78.74 127)
 		)
 		(stroke
@@
 			)
 			(justify left)
+		)
+	)
+	(text "Optional series resistor\n(or jumper wire)"
+		(exclude_from_sim no)
+		(at 77.47 123.19 0)
+		(effects
+			(font
+				(size 1.27 1.27)
+			)
+			(justify right)
 		)
 	)
@@
 					(unit 1)
 				)
+			)
+		)
+	)
+	(symbol
+		(lib_id "Device:R_US")
+		(at 78.74 123.19 180)
+		(unit 1)
+		(exclude_from_sim no)
+		(in_bom yes)
+		(on_board yes)
+		(dnp no)
+		(fields_autoplaced yes)
+		(property "Reference" "R4"
+			(at 81.28 123.1899 0)
+			(effects
+				(font
+					(size 1.27 1.27)
+				)
+				(justify right)
+			)
+		)
+		(property "Value" "10K"
+			(at 81.28 124.4599 0)
+			(effects
+				(font
+					(size 1.27 1.27)
+				)
+				(justify right)
+				(hide yes)
+			)
+		)
+		(property "Footprint" ""
+			(at 77.724 122.936 90)
+			(effects
+				(font
+					(size 1.27 1.27)
+				)
+				(hide yes)
+			)
+		)
+		(property "Datasheet" "~"
+			(at 78.74 123.19 0)
+			(effects
+				(font
+					(size 1.27 1.27)
+				)
+				(hide yes)
+			)
+		)
+		(property "Description" "Resistor, US symbol"
+			(at 78.74 123.19 0)
+			(effects
+				(font
+					(size 1.27 1.27)
+				)
+				(hide yes)
+			)
+		)
+		(pin "2"
+		)
+		(pin "1"
+		)
+		(instances
+			(project "busylight"
+				(path "/0c455002-a8fa-4df4-b787-466dd76b13a1"
+					(reference "R4")
+					(unit 1)
+				)
