File: hardware/ada/adashield.kicad_sch (KiCad schematic)
At the start: 33 parts, among them J1a Screw_Terminal_01x08, J1b RS-485 PASS-THRU, J3 RESET, J3 RESET DISABLE (Remove to prog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, J4 LOGIC VOLTAGE, J5 POWER, J6 SPEAKER, J7 LED Matrix, J8 Discrete LEDs, Q0 2N2222 / BC547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

Commit message: sync
Other:
- note added: "---------ROWS SELECTED------ E D C B A __ x 16 __ x 32 __ x 64 0 0 0 0 0 0 and 8 0 and 16 0 and 32 0 0 0 0 1 1 and 9 1 and 17 1 and 33 0 0 0 1 0 2 and 10 2 and 18 2 and 34 0 0 0 1 1 3 and 11 3 and 19 3 and 35 0 0 1 0 0 4 and 12 4 and 20 4 and 36 0 0 1 0 1 5 and 13 5 and 21 5 and 37 0 0 1 1 0 6 and 14 6 and 22 6 and 38 0 0 1 1 1 7 and 15 7 and 23 7 and 39 0 1 x x x 8,24-15,31 8,40-15,47 1 0 x x x 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"
Changed lines of the file:
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@@
+		)
+	)
+	(text "             ---------ROWS SELECTED------\nE D C B A    __ x 16    __ x 32    __ x 64\n0 0 0 0 0    0 and 8    0 and 16   0 and 32\n0 0 0 0 1    1 and 9    1 and 17   1 and 33\n0 0 0 1 0    2 and 10   2 and 18   2 and 34\n0 0 0 1 1    3 and 11   3 and 19   3 and 35\n0 0 1 0 0    4 and 12   4 and 20   4 and 36\n0 0 1 0 1    5 and 13   5 and 21   5 and 37\n0 0 1 1 0    6 and 14   6 and 22   6 and 38\n0 0 1 1 1    7 and 15   7 and 23   7 and 39\n0 1 x x x               8,24-15,31 8,40-15,47\n1 0 x x x                           16,48-23,55\n1 1 x x x                           24,56-31,63"
+		(exclude_from_sim no)
+		(at 85.09 152.4 0)
+		(effects
+			(font
+				(size 1.27 1.27)
+			)
+			(justify left top)
 		)
 	)
